Commit message: fix: meshes

File: ipa325_wsg50/urdf/wsg50.urdf.xacro (robot description, xacro)
@@ -16,5 +16,5 @@
                 <origin xyz="0 0 0" rpy="0 0 0" />
                 <geometry>
-                    <mesh filename="package://ipa325_robot_descriptions/meshes/tools/wsg50/WSG50_110.stl"/>
+                    <mesh filename="package://ipa325_wsg50/meshes/WSG50_110.stl"/>
                 </geometry>
                 <material name="wsg50-greyish">
@@ -25,5 +25,5 @@
                 <origin xyz="0 0 0" rpy="0 0 0" />
                 <geometry>
-                    <mesh filename="package://ipa325_robot_descriptions/meshes/tools/wsg50/WSG50_110.stl"/>
+                    <mesh filename="package://ipa325_wsg50/meshes/WSG50_110.stl"/>
                 </geometry>
             </collision>
