Commit message: xacro constant
use the provided constant, error when using this file standalone currently

File: weiss_wsg32_support/urdf/wsg32.urdf.xacro (robot description, xacro)
@@ -39,5 +39,5 @@
                 <parent link="${prefix}wsg_base_frame"/>
                 <child link="${prefix}finger_right_frame"/>
-                <origin xyz=" 0 0 0" rpy="0 0 ${m_pi}"/>
+                <origin xyz=" 0 0 0" rpy="0 0 ${pi}"/>
                 <axis xyz="0 -1 0"/>
                 <limit effort="0" lower="0" upper="0.05" velocity="0.001"/>

Commit message: Update wsg32.urdf.xacro

File: weiss_wsg32_support/urdf/wsg32.urdf.xacro (robot description, xacro)
@@ -2,5 +2,5 @@
 <robot xmlns:xacro="http://www.ros.org/wiki/xacro" name="wsg32">
     <xacro:macro name="wsg32" params="parent prefix *origin">
-        <joint name="{prefix}mount" type="fixed" >
+        <joint name="${prefix}mount" type="fixed" >
             <xacro:insert_block name="origin" />
             <parent link="${parent}" />
